Commit message: Push

File: autonomous_ws/src/msi_2k16_17_urdf/urdf/msi.xacro (robot description, xacro)
@@ -4,5 +4,6 @@
   <!-- <xacro:include filename="$(find husky_description)/urdf/decorations.urdf.xacro" /> -->
   <xacro:include filename="$(find msi_2k16_17_urdf)/urdf/wheel.urdf.xacro" />
-  <xacro:include filename="$(find msi_2k16_17_urdf)/urdf/arm.urdf" />
+  <xacro:include filename="$(find msi_2k16_17_urdf)/urdf/hokuyo.urdf.xacro" />
+  <!--<xacro:include filename="$(find msi_2k16_17_urdf)/urdf/arm.urdf" />-->
   <material name="chassis">
     <color rgba="0.67 0.78 0.85 1" />
@@ -219,3 +220,8 @@
         <origin xyz=" -0.2 0 0" rpy="0 0 ${M_PI}" />
       </joint>-->
+    <joint name="hokuyo_joint" type="fixed">
+      <origin xyz="0 0 0" rpy="0 0 0" />
+      <parent link="base_link" />
+      <child link="base_laser_link" />
+    </joint>
 </robot>

Commit message: Rover revamp

File: autonomous_ws/src/msi_2k16_17_urdf/urdf/msi.xacro (robot description, xacro)
@@ -4,5 +4,5 @@
   <!-- <xacro:include filename="$(find husky_description)/urdf/decorations.urdf.xacro" /> -->
   <xacro:include filename="$(find msi_2k16_17_urdf)/urdf/wheel.urdf.xacro" />
-  <xacro:include filename="$(find msi_2k16_17_urdf)/urdf/hokuyo.urdf.xacro" />
+  <!-- <xacro:include filename="$(find msi_2k16_17_urdf)/urdf/hokuyo.urdf.xacro" /> -->
   <!--<xacro:include filename="$(find msi_2k16_17_urdf)/urdf/arm.urdf" />-->
   <material name="chassis">
@@ -220,8 +220,9 @@
         <origin xyz=" -0.2 0 0" rpy="0 0 ${M_PI}" />
       </joint>-->
-    <joint name="hokuyo_joint" type="fixed">
+<!--     <joint name="hokuyo_joint" type="fixed">
       <origin xyz="0 0 0" rpy="0 0 0" />
       <parent link="base_link" />
       <child link="base_laser_link" />
     </joint>
+ -->
 </robot>
